File: omniBoard/omniBoard.sch (KiCad schematic (older format))
At the start: 21 parts, among them J2 Conn_01x02, J3 Conn_01x02, J4 Conn_01x04, J5 Conn_01x04, J6 Raspberry_Pi_2_3, J7 Conn_01x04, J8 Conn_01x04, U2 LM2596_module, U4 MPU6050_module

Commit message: Finish board 2nd version
Parts:
- added J1: Conn_01x02, TerminalBlock_Phoenix:TerminalBlock_Phoenix_MKDS-1,5-2-5.08_1x02_P5.08mm_Horizontal, symbol Connector_Generic:Conn_01x02
Connections:
- net +5V: now also J1.2 (Pin_2); no longer J6.2 (5V), J6.4 (5V)
- net GND: now also J1.1 (Pin_1)
- net _ENABLE: now also J6.10 (GPIO15/RXD)
- no-connect marks 4 -> 21
Other:
- moved on the sheet: C1, J2, J3, U2
Changed lines of the file:
@@
 	9850 1900 10300 1900
 Wire Wire Line
-	2500 4450 2500 4500
-Connection ~ 2500 4450
-Wire Wire Line
-	2650 4450 2500 4450
-Wire Wire Line
-	2650 4400 2650 4450
-Wire Wire Line
-	2500 4050 2500 4000
-Connection ~ 2500 4050
-Wire Wire Line
-	2650 4050 2500 4050
-Wire Wire Line
-	2650 4100 2650 4050
+	1800 4500 1800 4550
+Connection ~ 1800 4500
+Wire Wire Line
+	1950 4500 1800 4500
+Wire Wire Line
+	1950 4450 1950 4500
+Wire Wire Line
+	1800 4100 1800 4050
+Connection ~ 1800 4100
+Wire Wire Line
+	1950 4100 1800 4100
+Wire Wire Line
+	1950 4150 1950 4100
 $Comp
 L Device:CP C1
 U 1 1 61EF2CC8
-P 2650 4250
-F 0 "C1" V 2905 4250 50  0000 C CNN
-F 1 "220uF" V 2814 4250 50  0000 C CNN
-F 2 "Capacitor_THT:CP_Radial_D8.0mm_P3.50mm" H 2688 4100 50  0001 C CNN
-F 3 "~" H 2650 4250 50  0001 C CNN
-	1    2650 4250
+P 1950 4300
+F 0 "C1" V 2205 4300 50  0000 C CNN
+F 1 "220uF" V 2114 4300 50  0000 C CNN
+F 2 "Capacitor_THT:CP_Radial_D8.0mm_P3.50mm" H 1988 4150 50  0001 C CNN
+F 3 "~" H 1950 4300 50  0001 C CNN
+	1    1950 4300
 	1    0    0    -1
 $EndComp
@@
 L power:+12V #PWR03
 U 1 1 61D7A608
-P 2500 4000
-F 0 "#PWR03" H 2500 3850 50  0001 C CNN
-F 1 "+12V" H 2515 4173 50  0000 C CNN
-F 2 "" H 2500 4000 50  0001 C CNN
-F 3 "" H 2500 4000 50  0001 C CNN
-	1    2500 4000
-	1    0    0    -1
-$EndComp
-Wire Wire Line
-	2500 4200 2500 4050
-Wire Wire Line
-	2500 4300 2500 4450
+P 1800 4050
+F 0 "#PWR03" H 1800 3900 50  0001 C CNN
+F 1 "+12V" H 1815 4223 50  0000 C CNN
+F 2 "" H 1800 4050 50  0001 C CNN
+F 3 "" H 1800 4050 50  0001 C CNN
+	1    1800 4050
+	1    0    0    -1
+$EndComp
+Wire Wire Line
+	1800 4250 1800 4100
+Wire Wire Line
+	1800 4350 1800 4500
 $Comp
 L power:GND #PWR04
 U 1 1 61D7EA6F
-P 2500 4500
-F 0 "#PWR04" H 2500 4250 50  0001 C CNN
-F 1 "GND" H 2505 4327 50  0000 C CNN
-F 2 "" H 2500 4500 50  0001 C CNN
-F 3 "" H 2500 4500 50  0001 C CNN
-	1    2500 4500
-	1    0    0    -1
-$EndComp
-Wire Wire Line
-	3350 4450 3350 4550
-Wire Wire Line
-	3550 4550 3550 4450
+P 1800 4550
+F 0 "#PWR04" H 1800 4300 50  0001 C CNN
+F 1 "GND" H 1805 4377 50  0000 C CNN
+F 2 "" H 1800 4550 50  0001 C CNN
+F 3 "" H 1800 4550 50  0001 C CNN
+	1    1800 4550
+	1    0    0    -1
+$EndComp
+Wire Wire Line
+	2650 4500 2650 4600
+Wire Wire Line
+	2850 4600 2850 4500
 $Comp
 L power:GND #PWR012
 U 1 1 61D68436
-P 3550 4550
-F 0 "#PWR012" H 3550 4300 50  0001 C CNN
-F 1 "GND" H 3555 4377 50  0000 C CNN
-F 2 "" H 3550 4550 50  0001 C CNN
-F 3 "" H 3550 4550 50  0001 C CNN
-	1    3550 4550
-	1    0    0    -1
-$EndComp
-Wire Wire Line
-	3950 4050 3950 4000
-Wire Wire Line
-	3850 4050 3950 4050
+P 2850 4600
+F 0 "#PWR012" H 2850 4350 50  0001 C CNN
+F 1 "GND" H 2855 4427 50  0000 C CNN
+F 2 "" H 2850 4600 50  0001 C CNN
+F 3 "" H 2850 4600 50  0001 C CNN
+	1    2850 4600
+	1    0    0    -1
+$EndComp
+Wire Wire Line
+	3250 4100 3250 4050
+Wire Wire Line
+	3150 4100 3250 4100
 $Comp
 L power:+5V #PWR013
 U 1 1 61D3419A
-P 3950 4000
-F 0 "#PWR013" H 3950 3850 50  0001 C CNN
-F 1 "+5V" H 3965 4173 50  0000 C CNN
-F 2 "" H 3950 4000 50  0001 C CNN
-F 3 "" H 3950 4000 50  0001 C CNN
-	1    3950 4000
-	1    0    0    -1
-$EndComp
-Wire Wire Line
-	2950 4050 3050 4050
-Wire Wire Line
-	2950 4000 2950 4050
+P 3250 4050
+F 0 "#PWR013" H 3250 3900 50  0001 C CNN
+F 1 "+5V" H 3265 4223 50  0000 C CNN
+F 2 "" H 3250 4050 50  0001 C CNN
+F 3 "" H 3250 4050 50  0001 C CNN
+	1    3250 4050
+	1    0    0    -1
+$EndComp
+Wire Wire Line
+	2250 4100 2350 4100
+Wire Wire Line
+	2250 4050 2250 4100
 $Comp
 L power:+12V #PWR09
 U 1 1 61D30CB9
-P 2950 4000
-F 0 "#PWR09" H 2950 3850 50  0001 C CNN
-F 1 "+12V" H 2965 4173 50  0000 C CNN
-F 2 "" H 2950 4000 50  0001 C CNN
-F 3 "" H 2950 4000 50  0001 C CNN
-	1    2950 4000
+P 2250 4050
+F 0 "#PWR09" H 2250 3900 50  0001 C CNN
+F 1 "+12V" H 2265 4223 50  0000 C CNN
+F 2 "" H 2250 4050 50  0001 C CNN
+F 3 "" H 2250 4050 50  0001 C CNN
+	1    2250 4050
 	1    0    0    -1
 $EndComp
@@
 L power:GND #PWR011
 U 1 1 61D2C17F
-P 3350 4550
-F 0 "#PWR011" H 3350 4300 50  0001 C CNN
-F 1 "GND" H 3355 4377 50  0000 C CNN
-F 2 "" H 3350 4550 50  0001 C CNN
-F 3 "" H 3350 4550 50  0001 C CNN
-	1    3350 4550
+P 2650 4600
+F 0 "#PWR011" H 2650 4350 50  0001 C CNN
+F 1 "GND" H 2655 4427 50  0000 C CNN
+F 2 "" H 2650 4600 50  0001 C CNN
+F 3 "" H 2650 4600 50  0001 C CNN
+	1    2650 4600
 	1    0    0    -1
 $EndComp
@@
 L Connector_Generic:Conn_01x02 J2
 U 1 1 61CA8FB3
-P 1800 4300
-F 0 "J2" H 1800 3975 50  0000 C CNN
-F 1 "Conn_01x02" H 1850 4075 50  0000 C CNN
-F 2 "TerminalBlock_Phoenix:TerminalBlock_Phoenix_MKDS-1,5-2_1x02_P5.00mm_Horizontal" H 1800 4300 50  0001 C CNN
-F 3 "~" H 1800 4300 50  0001 C CNN
-	1    1800 4300
+P 1100 4350
+F 0 "J2" H 1100 4025 50  0000 C CNN
+F 1 "Conn_01x02" H 1150 4125 50  0000 C CNN
+F 2 "TerminalBlock_Phoenix:TerminalBlock_Phoenix_MKDS-1,5-2_1x02_P5.00mm_Horizontal" H 1100 4350 50  0001 C CNN
+F 3 "~" H 1100 4350 50  0001 C CNN
+	1    1100 4350
 	-1   0    0    1
 $EndComp
@@
 L omniBoard:LM2596_module U2
 U 1 1 61C9E104
-P 3450 4050
-F 0 "U2" H 3450 4315 50  0000 C CNN
-F 1 "LM2596_module" H 3450 4224 50  0000 C CNN
-F 2 "omniBoard:LM2596_module" H 3450 4050 50  0001 C CNN
-F 3 "" H 3450 4050 50  0001 C CNN
-	1    3450 4050
+P 2750 4100
+F 0 "U2" H 2750 4365 50  0000 C CNN
+F 1 "LM2596_module" H 2750 4274 50  0000 C CNN
+F 2 "omniBoard:LM2596_module" H 2750 4100 50  0001 C CNN
+F 3 "" H 2750 4100 50  0001 C CNN
+	1    2750 4100
 	1    0    0    -1
 $EndComp
@@
 	6100 2950 6150 2950
 $Comp
-L power:+5V #PWR0102
-U 1 1 61E0C81F
-P 5800 2900
-F 0 "#PWR0102" H 5800 2750 50  0001 C CNN
-F 1 "+5V" H 5815 3073 50  0000 C CNN
-F 2 "" H 5800 2900 50  0001 C CNN
-F 3 "" H 5800 2900 50  0001 C CNN
-	1    5800 2900
-	1    0    0    -1
-$EndComp
-Wire Wire Line
-	5800 2900 5800 2950
-Wire Wire Line
-	5800 2950 5850 2950
-Wire Wire Line
-	5850 2950 5850 3000
-Wire Wire Line
-	5800 2950 5750 2950
-Wire Wire Line
-	5750 2950 5750 3000
-Connection ~ 5800 2950
-$Comp
 L Connector_Generic:Conn_01x02 J3
 U 1 1 61D3D239
-P 2150 4000
-F 0 "J3" V 2350 4000 50  0000 R CNN
-F 1 "Conn_01x02" V 2250 4250 50  0000 R CNN
-F 2 "TerminalBlock_Phoenix:TerminalBlock_Phoenix_MKDS-1,5-2-5.08_1x02_P5.08mm_Horizontal" H 2150 4000 50  0001 C CNN
-F 3 "~" H 2150 4000 50  0001 C CNN
-	1    2150 4000
+P 1450 4050
+F 0 "J3" V 1650 4050 50  0000 R CNN
+F 1 "Conn_01x02" V 1550 4300 50  0000 R CNN
+F 2 "TerminalBlock_Phoenix:TerminalBlock_Phoenix_MKDS-1,5-2-5.08_1x02_P5.08mm_Horizontal" H 1450 4050 50  0001 C CNN
+F 3 "~" H 1450 4050 50  0001 C CNN
+	1    1450 4050
 	0    -1   -1   0
 $EndComp
 Wire Wire Line
-	2250 4200 2500 4200
-Wire Wire Line
-	2000 4300 2500 4300
-Wire Wire Line
-	2150 4200 2000 4200
+	1550 4250 1800 4250
+Wire Wire Line
+	1300 4350 1800 4350
+Wire Wire Line
+	1450 4250 1300 4250
 Text Label 7800 3400 2    50   ~ 0
 MS1
@@
 Wire Wire Line
 	5050 3800 5150 3800
+$Comp
+L Connector_Generic:Conn_01x02 J1
+U 1 1 61F61BFB
+P 4000 4350
+F 0 "J1" H 4000 4025 50  0000 C CNN
+F 1 "Conn_01x02" H 4050 4125 50  0000 C CNN
+F 2 "TerminalBlock_Phoenix:TerminalBlock_Phoenix_MKDS-1,5-2-5.08_1x02_P5.08mm_Horizontal" H 4000 4350 50  0001 C CNN
+F 3 "~" H 4000 4350 50  0001 C CNN
+	1    4000 4350
+	1    0    0    1
+$EndComp
+$Comp
+L power:+5V #PWR0105
+U 1 1 61FB2C74
+P 3700 4050
+F 0 "#PWR0105" H 3700 3900 50  0001 C CNN
+F 1 "+5V" H 3715 4223 50  0000 C CNN
+F 2 "" H 3700 4050 50  0001 C CNN
+F 3 "" H 3700 4050 50  0001 C CNN
+	1    3700 4050
+	1    0    0    -1
+$EndComp
+$Comp
+L power:GND #PWR0106
+U 1 1 61FB3726
+P 3700 4600
+F 0 "#PWR0106" H 3700 4350 50  0001 C CNN
+F 1 "GND" H 3705 4427 50  0000 C CNN
+F 2 "" H 3700 4600 50  0001 C CNN
+F 3 "" H 3700 4600 50  0001 C CNN
+	1    3700 4600
+	1    0    0    -1
+$EndComp
+Wire Wire Line
+	3800 4350 3700 4350
+Wire Wire Line
+	3700 4350 3700 4600
+Wire Wire Line
+	3800 4250 3700 4250
+Wire Wire Line
+	3700 4250 3700 4050
+NoConn ~ 5750 3000
+NoConn ~ 5850 3000
+NoConn ~ 6750 3400
+NoConn ~ 6750 3500
+NoConn ~ 5150 3400
+NoConn ~ 5150 4300
+NoConn ~ 5150 4500
+NoConn ~ 5150 4700
+NoConn ~ 5150 4800
+NoConn ~ 5150 4900
+NoConn ~ 5150 5000
+NoConn ~ 6750 4800
+NoConn ~ 6750 4700
+NoConn ~ 6750 4600
+NoConn ~ 6750 4500
+NoConn ~ 6750 4400
+NoConn ~ 6750 4100
+Text Label 5050 3500 2    50   ~ 0
+_ENABLE
+Wire Wire Line
+	5150 3500 5050 3500
 $EndSCHEMATC

Commit message: Add new led
Parts:
- added D2: LED, LED_THT:LED_D5.0mm, symbol Device:LED
- added R2: 68, Resistor_THT:R_Axial_DIN0207_L6.3mm_D2.5mm_P10.16mm_Horizontal, symbol Device:R
- R1: renamed from R7; value 330 -> 68
- renumbered J2 to J1, J3 to J2, J4 to J3, J1 to J4, U2 to U1, U4 to U2
Connections:
- net +3V3: now also R2.2
- net GND: now also D2.1 (K)
- new net: D2.2 (A), R2.1
Other:
- moved on the sheet: D1, R1

Commit message: Final version
Other:
- note added: "MOTORS AND\nDRIVERS\n"
- note added: "POWER"
- note added: "RASPBERRY"
- note added: "SENSOR AND\nINDICATORS"
- moved on the sheet: A1, A2, A3, A4, BZ1, C1, C2, C3, C4, C5, D1, D2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
